Commit message: Add kinematic and dynamic information

File: razbot_description/urdf/razbot.urdf.xacro (robot description, xacro)
@@ -14,5 +14,4 @@
   <xacro:property name="wheel_track" value="0.146" />
   <xacro:property name="wheel_vertical_offset" value="0" />
-  <xacro:property name="wheel_width" value="0.025" />
   <xacro:property name="wheel_width" value="0.025" />
   <xacro:property name="wheel_radius" value="0.040" />
@@ -47,4 +46,22 @@
       <material name="Blue" />
     </visual>
+    <!-- <collision> tags describe the collision boundaries of a link. You can use
+    the same contents as the <visual> tag. Even if you use a complex shape for the
+    <visual> tag, it's more efficient to use a basic bounding shape for collisions -->
+    <collision>
+      <origin xyz="0 0 0" rpy="0 0 0" />
+      <geometry>
+        <box size="${base_length} ${base_width} ${base_height}"/>
+      </geometry>
+    </collision>
+    <!-- <interial> tags describe intertial properties of the link. These are relative
+    to the origin of the link, so make sure the data you obtain is consistent -->
+    <inertial>
+      <origin xyz="0 0 0" />
+      <mass value="1.5" /> <!-- mass in kg -->
+      <inertia  ixx="0.01" ixy="0" ixz="0"
+                iyy="0.01" iyz="0"
+                izz="0.01" /> <!-- inertia around each axis pair -->
+    </inertial>
   </link>
   <!-- Xacro is an XML macro language that allows us to save effort when creating similar

File: razbot_description/urdf/wheel.urdf.xacro (robot description, xacro)
@@ -15,5 +15,37 @@
         <material name="Grey" />
       </visual>
+      <collision>
+        <origin xyz="0 0 0" rpy="${M_PI/2} 0 0" />
+        <geometry>
+          <cylinder length="${wheel_width}" radius="${wheel_radius}" />
+        </geometry>
+      </collision>
+      <inertial>
+        <origin xyz="0 0.1 0"/>
+        <mass value="0.15" />
+        <inertia  ixx="0.0001" ixy="0" ixz="0"
+                  iyy="0.0001" iyz="0"
+                  izz="0.0001" />
+      </inertial>
     </link>
+    <!-- This block provides the simulator (Gazebo) with information on a few additional
+    physical properties. See http://gazebosim.org/tutorials/?tut=ros_urdf for more-->
+    <gazebo reference="${wheel_prefix}_wheel_link">
+      <mu1 value="200.0"/>
+      <mu2 value="100.0"/>
+      <kp value="10000000.0" />
+      <kd value="1.0" />
+    </gazebo>
+    <!-- This block connects the wheel joint to an actuator (motor), which informs both
+    simulation and visualization of the robot -->
+    <transmission name="${wheel_prefix}_wheel_trans" type="SimpleTransmission">
+      <type>transmission_interface/SimpleTransmission</type>
+      <actuator name="${wheel_prefix}_wheel_motor">
+        <mechanicalReduction>1</mechanicalReduction>
+      </actuator>
+      <joint name="${wheel_prefix}_wheel">
+        <hardwareInterface>VelocityJointInterface</hardwareInterface>
+      </joint>
+    </transmission>
     <!-- Wheel to base joint. This joint is continuous so that the wheel can
     spin freely -->

Commit message: Create Gazebo bringup

File: razbot_description/urdf/razbot.urdf.xacro (robot description, xacro)
@@ -65,4 +65,7 @@
     </inertial>
   </link>
+  <gazebo reference="base_link">
+    <material>Gazebo/Blue</material>
+  </gazebo>
   <!-- Xacro is an XML macro language that allows us to save effort when creating similar
   XML blocks. Here, we create four wheels from the macro contained in the urdf/wheel.urdf.xacro

File: razbot_description/urdf/wheel.urdf.xacro (robot description, xacro)
@@ -36,4 +36,5 @@
       <kp value="10000000.0" />
       <kd value="1.0" />
+      <material>Gazebo/Grey</material>
     </gazebo>
     <!-- This block connects the wheel joint to an actuator (motor), which informs both

Commit message: Include STLs from SW for visualization

File: razbot_description/urdf/razbot.urdf.xacro (robot description, xacro)
@@ -42,5 +42,5 @@
       <origin xyz="0 0 0" rpy="0 0 0" />
       <geometry>
-        <box size="${base_length} ${base_width} ${base_height}"/>
+        <mesh filename="package://razbot_description/meshes/base.stl" />
       </geometry>
       <material name="Blue" />
@@ -72,14 +72,14 @@
   file -->
   <!-- Create wheels from macro -->
-  <xacro:razbot_wheel wheel_prefix="front_left">
+  <xacro:razbot_wheel wheel_prefix="front_left" flip="-1">
     <origin xyz="${wheel_base/2} ${wheel_track/2} ${wheel_vertical_offset}" rpy="0 0 0" />
   </xacro:razbot_wheel>
-  <xacro:razbot_wheel wheel_prefix="front_right">
+  <xacro:razbot_wheel wheel_prefix="front_right" flip="1">
     <origin xyz="${wheel_base/2} ${-wheel_track/2} ${wheel_vertical_offset}" rpy="0 0 0" />
   </xacro:razbot_wheel>
-  <xacro:razbot_wheel wheel_prefix="rear_left">
+  <xacro:razbot_wheel wheel_prefix="rear_left" flip="-1">
     <origin xyz="${-wheel_base/2} ${wheel_track/2} ${wheel_vertical_offset}" rpy="0 0 0" />
   </xacro:razbot_wheel>
-  <xacro:razbot_wheel wheel_prefix="rear_right">
+  <xacro:razbot_wheel wheel_prefix="rear_right" flip="1">
     <origin xyz="${-wheel_base/2} ${-wheel_track/2} ${wheel_vertical_offset}" rpy="0 0 0" />
   </xacro:razbot_wheel>

File: razbot_description/urdf/wheel.urdf.xacro (robot description, xacro)
@@ -5,11 +5,12 @@
   to the macro call, which can be simple parameters, or entire code blocks.
   See http://wiki.ros.org/xacro for more details. -->
-  <xacro:macro name="razbot_wheel" params="wheel_prefix *joint_pose">
+  <xacro:macro name="razbot_wheel" params="wheel_prefix flip *joint_pose">
     <!-- Wheel link -->
     <link name="${wheel_prefix}_wheel_link">
       <visual>
-        <origin xyz="0 0 0" rpy="${M_PI/2} 0 0" />
+        <!-- math-magic to get the wheel STLs to align -->
+        <origin xyz="${flip*wheel_radius} ${-flip*wheel_width/2} ${-wheel_radius}" rpy="${M_PI/2} 0 ${flip*M_PI/2+M_PI/2}" />
         <geometry>
-          <cylinder length="${wheel_width}" radius="${wheel_radius}" />
+          <mesh filename="package://razbot_description/meshes/wheel.stl" />
         </geometry>
         <material name="Grey" />

Commit message: Add intertial information from SW report

File: razbot_description/urdf/razbot.urdf.xacro (robot description, xacro)
@@ -59,8 +59,8 @@
     <inertial>
       <origin xyz="0 0 0" />
-      <mass value="1.5" /> <!-- mass in kg -->
-      <inertia  ixx="0.01" ixy="0" ixz="0"
-                iyy="0.01" iyz="0"
-                izz="0.01" /> <!-- inertia around each axis pair -->
+      <mass value="0.857" /> <!-- mass in kg -->
+      <inertia  ixx="2.17" ixy="0" ixz="0"
+                iyy="3.09" iyz="0"
+                izz="4.76" /> <!-- inertia around each axis pair -->
     </inertial>
   </link>

File: razbot_gazebo/urdf/razbot.gazebo.xacro (robot description, xacro)
@@ -25,3 +25,2 @@
   </gazebo>
 </robot>
-husky_v
